Commit message: Add UR5e + Robotiq 2F-85 MoveIt config (Phase 2)
Full MoveIt 2 config for the gripper-equipped arm, loading the combined
description into both ros2_control and move_group:
  - SRDF: reuses ur_srdf for the arm group, adds a gripper group with
    open/closed states, an end effector, and the 2F-85 self-collision disables.
  - kinematics (KDL), joint limits, ros2_controllers (joint_state_broadcaster,
    joint_trajectory_controller for the arm, position GripperActionController
    for the 2F-85), and the MoveIt controller bridge.
  - ur5e_gripper_moveit.launch.py brings it all up (RViz optional).

Uses the standard joint_trajectory_controller (the generic mock hardware has no
speed-scaling interface the UR scaled controller needs), and a minimal gripper
ros2_control driving only the active knuckle joint (mock rejects command
interfaces on mimic joints; robot_state_publisher derives the mimic fingers).

Verified headless (docs/phase2_gripper_verification.txt): arm plans and executes
via MoveIt (SUCCESS, within 0.009 rad) and the gripper opens/closes via its
GripperCommand action (reached_goal true).

File: ros2/src/armik_moveit/description/ur5e_robotiq.urdf.xacro (robot description, xacro)
@@ -34,5 +34,8 @@
   <xacro:include filename="$(find robotiq_description)/urdf/ur_to_robotiq_adapter.urdf.xacro"/>
   <xacro:ur_to_robotiq prefix="$(arg tf_prefix)" connected_to="$(arg tf_prefix)tool0"/>
-  <!-- Robotiq 2F-85 gripper (+ its own mock-hardware ros2_control) -->
+  <!-- Robotiq 2F-85 gripper links/joints only. Its bundled ros2_control block is
+       skipped (include_ros2_control=false): with mock hardware it puts command
+       interfaces on the mimic joints, which mock_components/GenericSystem rejects
+       ("activated mimic joints cannot have command interfaces"). -->
   <xacro:include filename="$(find robotiq_description)/urdf/robotiq_2f_85_macro.urdf.xacro"/>
   <xacro:robotiq_gripper
@@ -41,6 +44,21 @@
     parent="$(arg tf_prefix)gripper_mount_link"
     use_fake_hardware="true"
-    include_ros2_control="true">
+    include_ros2_control="false">
     <origin xyz="0 0 0" rpy="0 0 0"/>
   </xacro:robotiq_gripper>
+  <!-- Minimal gripper ros2_control: drive only the active knuckle joint. The
+       five mimic finger joints are computed by robot_state_publisher from the
+       URDF mimic tags, so they need no command/state interfaces here. -->
+  <ros2_control name="RobotiqGripper" type="system">
+    <hardware>
+      <plugin>mock_components/GenericSystem</plugin>
+    </hardware>
+    <joint name="$(arg tf_prefix)robotiq_85_left_knuckle_joint">
+      <command_interface name="position"/>
+      <state_interface name="position">
+        <param name="initial_value">0.0</param>
+      </state_interface>
+      <state_interface name="velocity"/>
+    </joint>
+  </ros2_control>
 </robot>
