Commit message: Mount the UR5e on a pedestal (industrial workcell layout)
Add a pedestal stand under the arm base (ur5e_robotiq.urdf.xacro, base raised
MOUNT_H=0.40 m) so the arm works downward over the cell from above, the standard
industrial palletizing layout. scene.py drops the whole cell by MOUNT_H into
base_link frame so it stays on the floor; the SRDF disables the base-on-pedestal
contact. Top-down reach from above is more natural, so planning is more reliable
(4/4, 0 re-plans, ~9.8 s/part) and the taller separator wall is comfortably
cleared.

File: ros2/src/armik_moveit/config/ur5e_robotiq.srdf.xacro (robot description, xacro)
@@ -12,4 +12,8 @@
   <xacro:include filename="$(find ur_moveit_config)/srdf/ur_macro.srdf.xacro"/>
   <xacro:ur_srdf/>
+  <!-- The arm base rests on the pedestal stand -->
+  <disable_collisions link1="pedestal" link2="base_link" reason="Adjacent"/>
+  <disable_collisions link1="pedestal" link2="base_link_inertia" reason="Adjacent"/>
+  <disable_collisions link1="pedestal" link2="shoulder_link" reason="Never"/>
   <!-- Gripper group: the single actuated knuckle joint drives the 2F-85 -->
   <group name="gripper">

File: ros2/src/armik_moveit/description/ur5e_robotiq.urdf.xacro (robot description, xacro)
@@ -14,6 +14,27 @@
   <xacro:arg name="ur_type" default="ur5e"/>
   <xacro:arg name="tf_prefix" default=""/>
+  <!-- The arm is mounted on a pedestal so it works downward over the cell from
+       above (the industrial workcell layout). base_link sits mount_h above the
+       floor; the cell geometry in scene.py is offset down by the same amount. -->
+  <xacro:property name="mount_h" value="0.40"/>
   <link name="world"/>
-  <!-- UR arm description -->
+  <!-- Pedestal stand from the floor up to the arm base -->
+  <link name="pedestal">
+    <visual>
+      <origin xyz="0 0 ${mount_h/2}" rpy="0 0 0"/>
+      <geometry><box size="0.20 0.20 ${mount_h}"/></geometry>
+      <material name="pedestal_gray"><color rgba="0.28 0.28 0.30 1"/></material>
+    </visual>
+    <collision>
+      <origin xyz="0 0 ${mount_h/2 - 0.01}" rpy="0 0 0"/>
+      <geometry><box size="0.20 0.20 ${mount_h - 0.02}"/></geometry>
+    </collision>
+  </link>
+  <joint name="world_to_pedestal" type="fixed">
+    <parent link="world"/>
+    <child link="pedestal"/>
+    <origin xyz="0 0 0" rpy="0 0 0"/>
+  </joint>
+  <!-- UR arm description, base raised onto the pedestal -->
   <xacro:include filename="$(find ur_description)/urdf/ur_macro.xacro"/>
   <xacro:ur_robot
@@ -26,5 +47,5 @@
     visual_parameters_file="$(find ur_description)/config/$(arg ur_type)/visual_parameters.yaml"
     safety_limits="true">
-    <origin xyz="0 0 0" rpy="0 0 0"/>
+    <origin xyz="0 0 ${mount_h}" rpy="0 0 0"/>
   </xacro:ur_robot>
   <!-- Arm ros2_control: mock hardware (mirrors command to state) -->
